Commit message: poprawki w launchfilach

File: urdf/afmer.urdf (robot description, URDF)
Before this commit: robot AFMER, 12 links, 11 joints
Joints:
- joint dummy_joint: origin (none) -> xyz=0 0 0

Commit message: tuning parametrow

File: urdf/afmer.urdf (robot description, URDF)
Before this commit: robot AFMER, 12 links, 11 joints
Links:
- removed link dummy
Joints:
- removed joint dummy_joint
- joint gear1_to_wheel1: type continuous -> fixed
- joint gear2_to_wheel2: type continuous -> fixed
- joint gear3_to_wheel3: type continuous -> fixed
- joint gear4_to_wheel4: type continuous -> fixed

Commit message: zmiana opisu robota

File: urdf/afmer.urdf (robot description, URDF)
Before this commit: robot AFMER, 11 links, 10 joints
Links:
- link base_link: geometry collision mesh filename=package://AFMER_description/models/AFMER/meshes/main.dae scale=1 1 1; visual mesh filename=package://AFMER_description/models/AFMER/meshes/main.dae scale=1 1 1
- link gear_1: geometry collision mesh filename=package://AFMER_description/models/AFMER/meshes/gearbox1.dae scale=1 1 1; visual mesh filename=package://AFMER_description/models/AFMER/meshes/gearbox1.dae scale=1 1 1
- link gear_2: geometry collision mesh filename=package://AFMER_description/models/AFMER/meshes/gearbox2.dae scale=1 1 1; visual mesh filename=package://AFMER_description/models/AFMER/meshes/gearbox2.dae scale=1 1 1
- link gear_3: geometry collision mesh filename=package://AFMER_description/models/AFMER/meshes/gearbox3.dae scale=1 1 1; visual mesh filename=package://AFMER_description/models/AFMER/meshes/gearbox3.dae scale=1 1 1
- link gear_4: geometry collision mesh filename=package://AFMER_description/models/AFMER/meshes/gearbox4.dae scale=1 1 1; visual mesh filename=package://AFMER_description/models/AFMER/meshes/gearbox4.dae scale=1 1 1
- link wheel_1: geometry collision mesh filename=package://AFMER_description/models/AFMER/meshes/wheel1.dae scale=1 1 1; visual mesh filename=package://AFMER_description/models/AFMER/meshes/wheel1.dae scale=1 1 1
- link wheel_2: geometry collision mesh filename=package://AFMER_description/models/AFMER/meshes/wheel2.dae scale=1 1 1; visual mesh filename=package://AFMER_description/models/AFMER/meshes/wheel2.dae scale=1 1 1
- link wheel_3: geometry collision mesh filename=package://AFMER_description/models/AFMER/meshes/wheel3.dae scale=1 1 1; visual mesh filename=package://AFMER_description/models/AFMER/meshes/wheel3.dae scale=1 1 1
- link wheel_4: geometry collision mesh filename=package://AFMER_description/models/AFMER/meshes/wheel4.dae scale=1 1 1; visual mesh filename=package://AFMER_description/models/AFMER/meshes/wheel4.dae scale=1 1 1

Commit message: Revert "zmiana opisu robota"
This reverts commit 6c2289ceaf01b693930a1bad3ae3f4d079abf204.

File: urdf/afmer.urdf (robot description, URDF)
Before this commit: robot AFMER, 11 links, 10 joints
Links:
- link base_link: geometry collision mesh filename=package://AFMER_description/models/AFMER/meshes/main.dae scale=0.001 0.001 0.001; visual mesh filename=package://AFMER_description/models/AFMER/meshes/main.dae scale=0.001 0.001 0.001
- link gear_1: geometry collision mesh filename=package://AFMER_description/models/AFMER/meshes/gearbox1.dae scale=0.001 0.001 0.001; visual mesh filename=package://AFMER_description/models/AFMER/meshes/gearbox1.dae scale=0.001 0.001 0.001
- link gear_2: geometry collision mesh filename=package://AFMER_description/models/AFMER/meshes/gearbox2.dae scale=0.001 0.001 0.001; visual mesh filename=package://AFMER_description/models/AFMER/meshes/gearbox2.dae scale=0.001 0.001 0.001
- link gear_3: geometry collision mesh filename=package://AFMER_description/models/AFMER/meshes/gearbox3.dae scale=0.001 0.001 0.001; visual mesh filename=package://AFMER_description/models/AFMER/meshes/gearbox3.dae scale=0.001 0.001 0.001
- link gear_4: geometry collision mesh filename=package://AFMER_description/models/AFMER/meshes/gearbox4.dae scale=0.001 0.001 0.001; visual mesh filename=package://AFMER_description/models/AFMER/meshes/gearbox4.dae scale=0.001 0.001 0.001
- link wheel_1: geometry collision mesh filename=package://AFMER_description/models/AFMER/meshes/wheel1.dae scale=0.001 0.001 0.001; visual mesh filename=package://AFMER_description/models/AFMER/meshes/wheel1.dae scale=0.001 0.001 0.001
- link wheel_2: geometry collision mesh filename=package://AFMER_description/models/AFMER/meshes/wheel2.dae scale=0.001 0.001 0.001; visual mesh filename=package://AFMER_description/models/AFMER/meshes/wheel2.dae scale=0.001 0.001 0.001
- link wheel_3: geometry collision mesh filename=package://AFMER_description/models/AFMER/meshes/wheel3.dae scale=0.001 0.001 0.001; visual mesh filename=package://AFMER_description/models/AFMER/meshes/wheel3.dae scale=0.001 0.001 0.001
- link wheel_4: geometry collision mesh filename=package://AFMER_description/models/AFMER/meshes/wheel4.dae scale=0.001 0.001 0.001; visual mesh filename=package://AFMER_description/models/AFMER/meshes/wheel4.dae scale=0.001 0.001 0.001

Commit message: skalowanie modelu

File: urdf/afmer.urdf (robot description, URDF)
Before this commit: robot AFMER, 11 links, 10 joints
Links:
- link imu_link: geometry visual box size=0.000312 0.000174 0.000022
- link laser: geometry visual cylinder length=0.0003 radius=0.00035

Commit message: powiekszenie robota

File: urdf/afmer.urdf (robot description, URDF)
Before this commit: robot AFMER, 11 links, 10 joints
Links:
- link base_link: geometry collision mesh filename=package://AFMER_description/models/AFMER/meshes/main.dae scale=0.1 0.1 0.1; visual mesh filename=package://AFMER_description/models/AFMER/meshes/main.dae scale=0.1 0.1 0.1
- link gear_1: geometry collision mesh filename=package://AFMER_description/models/AFMER/meshes/gearbox1.dae scale=0.1 0.1 0.1; visual mesh filename=package://AFMER_description/models/AFMER/meshes/gearbox1.dae scale=0.1 0.1 0.1
- link gear_2: geometry collision mesh filename=package://AFMER_description/models/AFMER/meshes/gearbox2.dae scale=0.1 0.1 0.1; visual mesh filename=package://AFMER_description/models/AFMER/meshes/gearbox2.dae scale=0.1 0.1 0.1
- link gear_3: geometry collision mesh filename=package://AFMER_description/models/AFMER/meshes/gearbox3.dae scale=0.1 0.1 0.1; visual mesh filename=package://AFMER_description/models/AFMER/meshes/gearbox3.dae scale=0.1 0.1 0.1
- link gear_4: geometry collision mesh filename=package://AFMER_description/models/AFMER/meshes/gearbox4.dae scale=0.1 0.1 0.1; visual mesh filename=package://AFMER_description/models/AFMER/meshes/gearbox4.dae scale=0.1 0.1 0.1
- link imu_link: geometry visual box size=0.0312 0.0174 0.0022
- link laser: geometry visual cylinder length=0.03 radius=0.035
- link wheel_1: geometry collision mesh filename=package://AFMER_description/models/AFMER/meshes/wheel1.dae scale=0.1 0.1 0.1; visual mesh filename=package://AFMER_description/models/AFMER/meshes/wheel1.dae scale=0.1 0.1 0.1
- link wheel_2: geometry collision mesh filename=package://AFMER_description/models/AFMER/meshes/wheel2.dae scale=0.1 0.1 0.1; visual mesh filename=package://AFMER_description/models/AFMER/meshes/wheel2.dae scale=0.1 0.1 0.1
- link wheel_3: geometry collision mesh filename=package://AFMER_description/models/AFMER/meshes/wheel3.dae scale=0.1 0.1 0.1; visual mesh filename=package://AFMER_description/models/AFMER/meshes/wheel3.dae scale=0.1 0.1 0.1
- link wheel_4: geometry collision mesh filename=package://AFMER_description/models/AFMER/meshes/wheel4.dae scale=0.1 0.1 0.1; visual mesh filename=package://AFMER_description/models/AFMER/meshes/wheel4.dae scale=0.1 0.1 0.1

Commit message: Kolejny resize

File: urdf/afmer.urdf (robot description, URDF)
Before this commit: robot AFMER, 11 links, 10 joints
Links:
- link base_link: geometry collision mesh filename=package://AFMER_description/models/AFMER/meshes/main.dae scale=0.01 0.01 0.01; visual mesh filename=package://AFMER_description/models/AFMER/meshes/main.dae scale=0.01 0.01 0.01
- link gear_1: geometry collision mesh filename=package://AFMER_description/models/AFMER/meshes/gearbox1.dae scale=0.01 0.01 0.01; visual mesh filename=package://AFMER_description/models/AFMER/meshes/gearbox1.dae scale=0.01 0.01 0.01
- link gear_2: geometry collision mesh filename=package://AFMER_description/models/AFMER/meshes/gearbox2.dae scale=0.01 0.01 0.01; visual mesh filename=package://AFMER_description/models/AFMER/meshes/gearbox2.dae scale=0.01 0.01 0.01
- link gear_3: geometry collision mesh filename=package://AFMER_description/models/AFMER/meshes/gearbox3.dae scale=0.01 0.01 0.01; visual mesh filename=package://AFMER_description/models/AFMER/meshes/gearbox3.dae scale=0.01 0.01 0.01
- link gear_4: geometry collision mesh filename=package://AFMER_description/models/AFMER/meshes/gearbox4.dae scale=0.01 0.01 0.01; visual mesh filename=package://AFMER_description/models/AFMER/meshes/gearbox4.dae scale=0.01 0.01 0.01
- link imu_link: geometry visual box size=0.00312 0.00174 0.00022
- link laser: geometry visual cylinder length=0.003 radius=0.0035
- link wheel_1: geometry collision mesh filename=package://AFMER_description/models/AFMER/meshes/wheel1.dae scale=0.01 0.01 0.01; visual mesh filename=package://AFMER_description/models/AFMER/meshes/wheel1.dae scale=0.01 0.01 0.01
- link wheel_2: geometry collision mesh filename=package://AFMER_description/models/AFMER/meshes/wheel2.dae scale=0.01 0.01 0.01; visual mesh filename=package://AFMER_description/models/AFMER/meshes/wheel2.dae scale=0.01 0.01 0.01
- link wheel_3: geometry collision mesh filename=package://AFMER_description/models/AFMER/meshes/wheel3.dae scale=0.01 0.01 0.01; visual mesh filename=package://AFMER_description/models/AFMER/meshes/wheel3.dae scale=0.01 0.01 0.01
- link wheel_4: geometry collision mesh filename=package://AFMER_description/models/AFMER/meshes/wheel4.dae scale=0.01 0.01 0.01; visual mesh filename=package://AFMER_description/models/AFMER/meshes/wheel4.dae scale=0.01 0.01 0.01
